File: Kicad/Mouse module 2.sch (KiCad schematic (older format))
At the start: 29 parts, among them J1 Conn_02x20_Odd_Even, J2 02x08_IDC, J3 TRIG, J4 X, J5 Y, J6 GATE, U1 TL074

Commit message: general cleanup & dual TL072
Parts:
- removed U1: TL074, symbol Amplifier_Operational:TL074
- added C?: 0.1uF, Capacitor_THT:C_Disc_D4.7mm_W2.5mm_P5.00mm, symbol Device:C_Small
- added C? (x2): 1uF, symbol Device:CP_Small
- added U1, U2: TL072, symbol Amplifier_Operational:TL072
Connections:
- wire segments 129 -> 147
Other:
- moved on the sheet: C1, C2, C3, C4, C5, C6, J3, J4, J5, J6, R1, R10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

Commit message: work on PCB & added some LEDs
Parts:
- removed J6: GATE, SJ1-3533:CUI_SJ1-3533, symbol Connector:AudioJack3
- removed unit 1 of U1
- removed unit 2 of U2
- removed unit 3 of U2
- added C?: 2.2u, Capacitor_THT:C_Disc_D4.7mm_W2.5mm_P5.00mm, symbol Device:C_Small
- added D?: GATE_LED, symbol Device:LED_Small
- added D?: TRIG_LED, symbol Device:LED_Small
- added D?: REC_LED, symbol Device:LED_Small
- added J3: GATE, MouseModule:CUI_SJ1-3533, symbol Connector:AudioJack3
- added R? (x2): 180, symbol Device:R_Small
- added R?: 180, Resistor_THT:R_Axial_DIN0207_L6.3mm_D2.5mm_P10.16mm_Horizontal, symbol Device:R_Small
- added U2: LM393, Package_DIP:DIP-8_W7.62mm, symbol Comparator:LM393
- C1, C2: renamed from C?; value 1uF -> 1u; footprint (none) -> Capacitor_THT:CP_Radial_D10.0mm_P5.00mm
- C3: value 0.1uF -> 0.1u
- C4: renamed from C5; value 0.1uF -> 0.1u
- C5: renamed from C?; value 0.1uF -> 0.1u
- C6: renamed from C1; value 0.1uF -> 0.1u
- C7: renamed from C2; value 0.1uF -> 0.1u
- C8: renamed from C4; value 0.1uF -> 0.1u
- C9: renamed from C6; value 0.1uF -> 0.1u
- J4, J5: footprint SJ1-3533:CUI_SJ1-3533 -> MouseModule:CUI_SJ1-3533
- J6: renamed from J3; footprint SJ1-3533:CUI_SJ1-3533 -> MouseModule:CUI_SJ1-3533
- U1: renamed from U2; footprint (none) -> Package_DIP:DIP-8_W7.62mm
- U1: footprint (none) -> Package_DIP:DIP-8_W7.62mm
- renumbered R3 to R1, R4 to R2, R1 to R3, R2 to R4
Connections:
- net +5V: now also U2.8 (V+)
- net GND: now also C?.1, J3.S, R?.1, R?.2, R?.2, U2.4 (V-)
- net RB_GATE: now also U2.3 (+); no longer U1.3 (+)
- net RB_TRIG: now also U2.5 (+)
- net at J1.7 (Pin_7): now also D?.2 (A)
- net at J4.T, R13.1: now also U1.1
- net at R7.1, R9.2: now also U1.3 (+)
- net at R11.2, R13.2: now also U1.2 (-)
- net at R3.1, R4.2: now also U2.2 (-); no longer U1.2 (-)
- net at R15.1, R16.2: now also U2.6 (_)
- net at J6.T: now also D?.2 (A), U2.7
- new net: D?.2 (A), J3.T, U2.1
- new net: D?.1 (K), R?.1 (x2)
- new net: C?.2, D?.1 (K), R?.2
- no-connect marks 37 -> 36
Other:
- moved on the sheet: U1A
