File: Kicad/Mouse module 2.kicad_pcb (KiCad board)
At the start: 2 copper layers, 67 x 65 mm, 29 parts, among them J1 Conn_02x20_Odd_Even, J2 02x08_IDC, J3 AudioJack3, J4 AudioJack3, J5 AudioJack3, J6 AudioJack3, J7 AudioJack3, U1 74LS125, U2 TL072, U3 MCP4922

Commit message: work on PCB & added some LEDs
Parts:
- removed H1, H2, H3, H4: MountingHole_Pad, MountingHole:MountingHole_2.7mm_Pad
- removed J7: AudioJack3, SJ1-3533:CUI_SJ1-3533
- removed U3: MCP4922, Package_DIP:DIP-14_W7.62mm_Socket
- added C6: 0.1uF, Capacitor_THT:C_Disc_D4.7mm_W2.5mm_P5.00mm, F.Cu at (45.4, 70.5)
- added C7: 0.1uF, Capacitor_THT:C_Disc_D4.7mm_W2.5mm_P5.00mm, F.Cu at (48.0, 37.5)
- added C8: 0.1uF, Capacitor_THT:C_Disc_D4.7mm_W2.5mm_P5.00mm, F.Cu at (67.0, 52.5)
- added C9: 0.1uF, Capacitor_THT:C_Disc_D4.7mm_W2.5mm_P5.00mm, F.Cu at (66.7, 39.4)
- added R11: 15k, Resistor_THT:R_Axial_DIN0207_L6.3mm_D2.5mm_P10.16mm_Horizontal, F.Cu at (30.2, 50.2)
- added R12: 15k, Resistor_THT:R_Axial_DIN0207_L6.3mm_D2.5mm_P10.16mm_Horizontal, F.Cu at (25.2, 22.9)
- added R13: 37k, Resistor_THT:R_Axial_DIN0207_L6.3mm_D2.5mm_P10.16mm_Horizontal, F.Cu at (26.7, 50.2)
- added R14: 37k, Resistor_THT:R_Axial_DIN0207_L6.3mm_D2.5mm_P10.16mm_Horizontal, F.Cu at (25.2, 26.1)
- added R15: 10k, Resistor_THT:R_Axial_DIN0207_L6.3mm_D2.5mm_P10.16mm_Horizontal, F.Cu at (38.4, 58.0)
- added R16: 4.7k, Resistor_THT:R_Axial_DIN0207_L6.3mm_D2.5mm_P10.16mm_Horizontal, F.Cu at (28.3, 61.2)
- added REF**: CE-Logo_8.5x6mm_SilkScreen, Symbol:CE-Logo_8.5x6mm_SilkScreen, F.Cu at (82.7, 139.2)
- added REF**: CE-Logo_8.5x6mm_SilkScreen, Symbol:CE-Logo_8.5x6mm_SilkScreen, F.Cu at (82.7, 110.0)
- C1: value 0.1uF -> 1uF; footprint Capacitor_THT:C_Disc_D4.7mm_W2.5mm_P5.00mm -> Capacitor_THT:CP_Radial_D10.0mm_P5.00mm
- C2: value 10uF -> 1uF; footprint Capacitor_THT:C_Disc_D4.7mm_W2.5mm_P5.00mm -> Capacitor_THT:CP_Radial_D10.0mm_P5.00mm
- J1: moved to F.Cu
- J3: value AudioJack3 -> GATE; footprint SJ1-3533:CUI_SJ1-3533 -> MouseModule:CUI_SJ1-3533
- J4: value AudioJack3 -> X; footprint SJ1-3533:CUI_SJ1-3533 -> MouseModule:CUI_SJ1-3533
- J5: value AudioJack3 -> Y; footprint SJ1-3533:CUI_SJ1-3533 -> MouseModule:CUI_SJ1-3533
- J6: value AudioJack3 -> TRIG; footprint SJ1-3533:CUI_SJ1-3533 -> MouseModule:CUI_SJ1-3533
- R1: value 2.7k -> 10k
- R10, R9: value 5.6k -> 150k
- R2: value 5.6k -> 10k
- R3: value 33k -> 10k
- R4: value 6.8k -> 4.7k
- R5: value 3.9k -> 10k
- R6: value 6.8k -> 10k
- R7: value 3.9k -> 670
- R8: value 33k -> 670
- U1: value 74LS125 -> TL072; footprint Package_DIP:DIP-14_W7.62mm_Socket -> Package_DIP:DIP-8_W7.62mm
- U2: value TL072 -> LM393; footprint Package_DIP:DIP-8_W7.62mm_Socket -> Package_DIP:DIP-8_W7.62mm
- moved C1 57.7 mm to (39.4, 126.2), turned to 90 degrees
- moved C5 51.4 mm to (26.9, 70.2), turned to 90 degrees
- moved J3 44.8 mm to (85.5, 76.4)
- moved R1 42.2 mm to (45.4, 61.8), turned to 0 degrees
- moved U2 41.0 mm to (30.3, 71.6), turned to 90 degrees
- moved R3 40.8 mm to (23.5, 73.0), turned to 90 degrees
- moved C4 36.0 mm to (23.1, 35.4), turned to 90 degrees
- moved R5 34.3 mm to (55.6, 58.3), turned to 180 degrees
- moved R7 31.4 mm to (45.4, 54.9)
- moved J2 29.0 mm to (25.3, 105.8), turned to 0 degrees
- moved R4 27.6 mm to (38.5, 74.5), turned to 180 degrees
- moved R6 25.3 mm to (55.6, 47.9), turned to 180 degrees
- moved U1 25.0 mm to (26.6, 36.7), turned to 90 degrees
- moved R2 24.8 mm to (45.4, 51.4), turned to 0 degrees
- moved C2 24.3 mm to (27.8, 83.5), turned to 270 degrees
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Connections:
- C1 pad 1: GND -> +12V
- C1 pad 2: +5V -> GND
- C2 pad 2: +5V -> -12V
- C4 pad 2: +5V -> +12V
- C5 pad 2: +12V -> +5V
- J1 pad 12: Net-(J1-Pad12) -> RB_X
- J1 pad 19: GPIO10(MOSI) -> Net-(J1-Pad19)
- J1 pad 23: GPIO11(SCLK) -> Net-(J1-Pad23)
- J1 pad 29: GPIO5 -> RB_GATE
- J1 pad 31: GPIO6 -> RB_TRIG
- J1 pad 33: Net-(J1-Pad33) -> RB_Y
- J1 pad 37: GPIO26 -> Net-(J1-Pad37)
- J4 pad T: CV_X -> Net-(J4-PadT)
- J5 pad T: CV_Y -> Net-(J5-PadT)
- J6 pad T: GATE -> Net-(J6-PadT)
- R1 pad 1: GPIO26 -> Net-(C6-Pad2)
- R1 pad 2: Net-(J3-PadT) -> RB_X
- R10 pad 1: CV_Y -> -12V
- R2 pad 1: GND -> Net-(C7-Pad2)
- R2 pad 2: GPIO26 -> RB_Y
- R3 pad 2: -12V -> +5V
- R4 pad 1: Net-(R4-Pad1) -> GND
- R5 pad 1: Net-(R5-Pad1) -> Net-(C8-Pad2)
- R5 pad 2: GND -> Net-(C6-Pad2)
- R6 pad 1: Net-(R6-Pad1) -> Net-(C9-Pad2)
- R6 pad 2: Net-(R6-Pad2) -> Net-(C7-Pad2)
- R7 pad 1: Net-(R10-Pad2) -> Net-(R7-Pad1)
- R7 pad 2: GND -> Net-(C8-Pad2)
- R8 pad 1: -12V -> Net-(R10-Pad2)
- R8 pad 2: Net-(R6-Pad1) -> Net-(C9-Pad2)
- R9 pad 1: CV_X -> -12V
- R9 pad 2: Net-(R5-Pad1) -> Net-(R7-Pad1)
- U1 pad 1: GND -> Net-(J4-PadT)
- U1 pad 2: GPIO11(SCLK) -> Net-(R11-Pad2)
- U1 pad 3: SCK -> Net-(R7-Pad1)
- U1 pad 4: GND -> -12V
- U1 pad 5: GPIO10(MOSI) -> Net-(R10-Pad2)
- U1 pad 6: SDI -> Net-(R12-Pad2)
- U1 pad 7: GND -> Net-(J5-PadT)
- U1 pad 8: GATE -> +12V
- U2 pad 1: CV_X -> Net-(J3-PadT)
- U2 pad 2: Net-(R5-Pad1) -> Net-(R3-Pad1)
- U2 pad 3: Net-(R6-Pad1) -> RB_GATE
- U2 pad 4: -12V -> GND
- U2 pad 5: Net-(R3-Pad1) -> RB_TRIG
- U2 pad 6: Net-(R10-Pad2) -> Net-(R15-Pad1)
- U2 pad 7: CV_Y -> Net-(J6-PadT)
- U2 pad 8: +12V -> +5V
Routing:
- net +5V: track 82.5 -> 15.2 mm
- net CV_X: track 56.7 -> 0.00 mm
- net +12V: track 52.7 -> 3.97 mm
- net -12V: track 48.2 -> 4.49 mm
- net CV_Y: track 42.5 -> 0.00 mm
- net TRIG: track 34.0 -> 0.00 mm
- net GATE: track 29.3 -> 0.00 mm
- net GPIO5: track 27.7 -> 0.00 mm
- net Net-(R6-Pad1): track 23.3 -> 0.00 mm
- net Net-(R10-Pad2): track 26.3 -> 3.46 mm
- net GPIO6: track 21.4 -> 0.00 mm
- net GPIO10(MOSI): track 17.5 -> 0.00 mm
- net Net-(C7-Pad2): track 0.00 -> 17.0 mm
- net GPIO11(SCLK): track 16.5 -> 0.00 mm
- net Net-(J3-PadT): track 14.5 -> 0.00 mm
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Other:
- board size 67 x 65 mm -> 67 x 110 mm

Commit message: update KiCad version
Other:
- net class Default removed
